File: OTTO-main/OTTO-main.kicad_pcb (KiCad board)
At the start: 2 copper layers, 239 x 76.4 mm, 16 parts, among them J1 Raspberry_Pi_2_3, J2 POWER_BOARD, J3 AUDIO_BOARD, J4 MICROPHONE, U1 STM32F103CBTx, Y1 8mhz

Commit message: some progress on the main board design
Parts:
- removed the REF** at (263.2, 37.3)
- removed the REF** at (147.7, 105.7)
- removed the REF** at (32.2, 105.7)
- removed the REF** at (32.2, 37.3)
- added C4: 1uf, Capacitor_SMD:C_0805_2012Metric, F.Cu at (-24.8, 160.8)
- added C5: 10nf, Capacitor_SMD:C_0805_2012Metric, F.Cu at (-24.8, 155.8)
- added D1: D_ALT, Diode_SMD:D_SOD-123, B.Cu at (242.8, 62.7)
- added D10: D_ALT, Diode_SMD:D_SOD-123, B.Cu at (47.0, 75.8)
- added D11: D_ALT, Diode_SMD:D_SOD-123, B.Cu at (59.6, 75.8)
- added D12: D_ALT, Diode_SMD:D_SOD-123, B.Cu at (72.2, 75.8)
- added D13: D_ALT, Diode_SMD:D_SOD-123, B.Cu at (84.8, 75.8)
- added D14: D_ALT, Diode_SMD:D_SOD-123, B.Cu at (97.5, 75.8)
- added D15: D_ALT, Diode_SMD:D_SOD-123, B.Cu at (110.0, 75.8)
- added D16: D_ALT, Diode_SMD:D_SOD-123, B.Cu at (122.7, 75.8)
- added D17: D_ALT, Diode_SMD:D_SOD-123, B.Cu at (34.5, 91.9)
- added D18: D_ALT, Diode_SMD:D_SOD-123, B.Cu at (47.0, 91.9)
- added D19: D_ALT, Diode_SMD:D_SOD-123, B.Cu at (59.6, 91.9)
- added D2: D_ALT, Diode_SMD:D_SOD-123, B.Cu at (255.4, 62.7)
- added D20: D_ALT, Diode_SMD:D_SOD-123, B.Cu at (72.2, 91.9)
- added D21: D_ALT, Diode_SMD:D_SOD-123, B.Cu at (84.8, 91.9)
- added D22: D_ALT, Diode_SMD:D_SOD-123, B.Cu at (97.5, 91.9)
- added D23: D_ALT, Diode_SMD:D_SOD-123, B.Cu at (110.0, 91.9)
- added D24: D_ALT, Diode_SMD:D_SOD-123, B.Cu at (122.7, 91.9)
- added D25: D_ALT, Diode_SMD:D_SOD-123, B.Cu at (135.2, 91.9)
- added D26: D_ALT, Diode_SMD:D_SOD-123, B.Cu at (135.2, 75.8)
- added D3: D_ALT, Diode_SMD:D_SOD-123, B.Cu at (242.8, 78.8)
- added D4: D_ALT, Diode_SMD:D_SOD-123, B.Cu at (255.4, 78.8)
- added D5: D_ALT, Diode_SMD:D_SOD-123, B.Cu at (242.8, 94.9)
- added D6: D_ALT, Diode_SMD:D_SOD-123, B.Cu at (255.4, 94.9)
- added D7: D_ALT, Diode_SMD:D_SOD-123, B.Cu at (34.5, 43.6)
- added D8: D_ALT, Diode_SMD:D_SOD-123, B.Cu at (34.5, 59.7)
- added D9: D_ALT, Diode_SMD:D_SOD-123, B.Cu at (34.5, 75.8)
- added L1: 30ohm, Capacitor_SMD:C_0805_2012Metric, F.Cu at (-24.8, 165.8)
- added REF**: MountingHole_3.2mm_M3, MountingHole:MountingHole_3.2mm_M3, F.Cu at (260.4, 38.5)
- added REF**: MountingHole_3.2mm_M3, MountingHole:MountingHole_3.2mm_M3, F.Cu at (144.9, 110.5)
- added REF**: MountingHole_3.2mm_M3, MountingHole:MountingHole_3.2mm_M3, F.Cu at (143.9, 38.5)
- added SW1: SW_SPST, Button_Switch_THT:Tactile_Switch_12x12x7.3_mm, F.Cu at (242.8, 62.7)
- added SW10: SW_SPST, Button_Switch_THT:Tactile_Switch_12x12x7.3_mm, F.Cu at (47.0, 75.8)
- added SW11: SW_SPST, Button_Switch_THT:Tactile_Switch_12x12x7.3_mm, F.Cu at (59.6, 75.8)
- added SW12: SW_SPST, Button_Switch_THT:Tactile_Switch_12x12x7.3_mm, F.Cu at (72.2, 75.8)
- added SW13: SW_SPST, Button_Switch_THT:Tactile_Switch_12x12x7.3_mm, F.Cu at (84.8, 75.8)
- added SW14: SW_SPST, Button_Switch_THT:Tactile_Switch_12x12x7.3_mm, F.Cu at (97.5, 75.8)
- added SW15: SW_SPST, Button_Switch_THT:Tactile_Switch_12x12x7.3_mm, F.Cu at (110.0, 75.8)
- added SW16: SW_SPST, Button_Switch_THT:Tactile_Switch_12x12x7.3_mm, F.Cu at (122.7, 75.8)
- added SW17: SW_SPST, Button_Switch_THT:Tactile_Switch_12x12x7.3_mm, F.Cu at (34.5, 91.9)
- added SW18: SW_SPST, Button_Switch_THT:Tactile_Switch_12x12x7.3_mm, F.Cu at (47.0, 91.9)
- added SW19: SW_SPST, Button_Switch_THT:Tactile_Switch_12x12x7.3_mm, F.Cu at (59.6, 91.9)
- added SW2: SW_SPST, Button_Switch_THT:Tactile_Switch_12x12x7.3_mm, F.Cu at (255.4, 62.7)
- added SW20: SW_SPST, Button_Switch_THT:Tactile_Switch_12x12x7.3_mm, F.Cu at (72.2, 91.9)
- added SW21: SW_SPST, Button_Switch_THT:Tactile_Switch_12x12x7.3_mm, F.Cu at (84.8, 91.9)
- added SW22: SW_SPST, Button_Switch_THT:Tactile_Switch_12x12x7.3_mm, F.Cu at (97.5, 91.9)
- added SW23: SW_SPST, Button_Switch_THT:Tactile_Switch_12x12x7.3_mm, F.Cu at (110.0, 91.9)
- added SW24: SW_SPST, Button_Switch_THT:Tactile_Switch_12x12x7.3_mm, F.Cu at (122.7, 91.9)
- added SW25: SW_SPST, Button_Switch_THT:Tactile_Switch_12x12x7.3_mm, F.Cu at (135.2, 91.9)
- added SW26: SW_SPST, Button_Switch_THT:Tactile_Switch_12x12x7.3_mm, F.Cu at (135.2, 75.8)
- added SW3: SW_SPST, Button_Switch_THT:Tactile_Switch_12x12x7.3_mm, F.Cu at (242.8, 78.8)
- added SW4: SW_SPST, Button_Switch_THT:Tactile_Switch_12x12x7.3_mm, F.Cu at (255.4, 78.8)
- added SW5: SW_SPST, Button_Switch_THT:Tactile_Switch_12x12x7.3_mm, F.Cu at (242.8, 94.9)
- added SW6: SW_SPST, Button_Switch_THT:Tactile_Switch_12x12x7.3_mm, F.Cu at (255.4, 94.9)
- added SW7: SW_SPST, Button_Switch_THT:Tactile_Switch_12x12x7.3_mm, F.Cu at (34.5, 43.6)
- added SW8: SW_SPST, Button_Switch_THT:Tactile_Switch_12x12x7.3_mm, F.Cu at (34.5, 59.7)
- added SW9: SW_SPST, Button_Switch_THT:Tactile_Switch_12x12x7.3_mm, F.Cu at (34.5, 75.8)
- moved U1 224.6 mm to (-49.9, 162.8), turned to 225 degrees
- moved C1 224.4 mm to (-60.5, 159.8)
- moved C2 224.4 mm to (-60.5, 162.6)
- moved C3 224.4 mm to (-60.5, 165.3)
- moved C6 224.4 mm to (-34.0, 164.1)
- moved C7 224.4 mm to (-34.0, 161.0)
- moved Y1 224.4 mm to (-40.0, 162.6)
- moved J3 147.9 mm to (102.1, 106.4), turned to 270 degrees
- moved REF** 97.8 mm to (49.0, 38.5)
- moved J4 6.72 mm to (260.6, 108.0)
- moved J2 6.03 mm to (228.2, 68.5)
- moved J1 3.00 mm to (151.4, 37.0)
- renumbered C4 to C2, C5 to C3, C2 to C6, C3 to C7, J2 to J1, J3 to J2, J1 to J3
Connections:
- net Net-(C1-Pad1) renamed +3V3
- net Net-(U1-Pad20) renamed BOOT1
- net Net-(U1-Pad7) renamed NRST
- J3 pad 10: Net-(J1-Pad10) -> UART_RXD
- J3 pad 15: Net-(J1-Pad15) -> OUT_PIN
- J3 pad 16: Net-(J1-Pad16) -> SENSE_PIN
- J3 pad 18: Net-(J1-Pad18) -> LED_G
- J3 pad 22: Net-(J1-Pad22) -> LED_R
- J3 pad 8: Net-(J1-Pad8) -> UART_TXD
- U1 pad 30: Net-(U1-Pad30) -> UART_RXD
- U1 pad 31: Net-(U1-Pad31) -> UART_TXD
- U1 pad 44: Net-(U1-Pad44) -> GNDREF
Other:
- board size 239 x 76.4 mm -> 239 x 80 mm
- rule trace_min: 0.2 -> 0.18
