File: OTTO-main/OTTO-main.kicad_pcb (KiCad board)
At the start: 2 copper layers, 239 x 80 mm, 70 parts, among them J1 POWER_BOARD, J2 AUDIO_BOARD, J3 Raspberry_Pi_2_3, J4 MICROPHONE, SW1 SW_SPST, SW10 SW_SPST, SW11 SW_SPST, SW12 SW_SPST, SW13 SW_SPST, SW14 SW_SPST, SW15 SW_SPST, SW16 SW_SPST, SW17 SW_SPST, SW18 SW_SPST, SW19 SW_SPST, SW2 SW_SPST, SW20 SW_SPST, SW21 SW_SPST, SW22 SW_SPST, SW23 SW_SPST, SW24 SW_SPST, SW25 SW_SPST, SW26 SW_SPST, SW3 SW_SPST, SW4 SW_SPST, SW5 SW_SPST, SW6 SW_SPST, SW7 SW_SPST, SW8 SW_SPST, SW9 SW_SPST, U1 STM32F103CBTx, Y1 8mhz

Commit message: mainboard
Parts:
- added C1: 10uf, Capacitor_Tantalum_SMD:CP_EIA-3216-18_Kemet-A, F.Cu at (171.9, 27.4)
- added C10: 0.1uF, Capacitor_SMD:C_0805_2012Metric, F.Cu at (-24.3, 31.8)
- added C11: 0.1uF, Capacitor_SMD:C_0805_2012Metric, F.Cu at (-67.2, 75.1)
- added C12: 0.1uF, Capacitor_SMD:C_0805_2012Metric, F.Cu at (-60.8, 69.3)
- added C13: 0.1uF, Capacitor_SMD:C_0805_2012Metric, F.Cu at (-70.6, 76.0)
- added C14: 0.1uF, Capacitor_SMD:C_0805_2012Metric, F.Cu at (-78.4, 78.6)
- added C2: 22uf, Capacitor_Tantalum_SMD:CP_EIA-3216-18_Kemet-A, F.Cu at (159.4, 27.4)
- added D1: 1N4148, Diode_SMD:D_SOD-123v, F.Cu at (-71.2, 72.7)
- added D2: 1N4148, Diode_SMD:D_SOD-123v, F.Cu at (-36.1, 40.5)
- added D3: 1N4148, Diode_SMD:D_SOD-123v, F.Cu at (-63.7, 68.8)
- added D4: 1N4148, Diode_SMD:D_SOD-123v, F.Cu at (-27.2, 33.2)
- added IC1: 74HC125, Package_SO:SOIC-14_3.9x8.7mm_P1.27mm, F.Cu at (-68.6, 65.6)
- added R1: 4.7K, Resistor_SMD:R_0805_2012Metric, F.Cu at (-68.3, 73.2)
- added R10: 10K, Resistor_SMD:R_0805_2012Metric, F.Cu at (-30.9, 42.9)
- added R11: 10K, Resistor_SMD:R_0805_2012Metric, F.Cu at (-67.2, 77.1)
- added R12: 10K, Resistor_SMD:R_0805_2012Metric, F.Cu at (-55.7, 65.8)
- added R13: 1.5K, Resistor_SMD:R_0805_2012Metric, F.Cu at (-40.5, 50.9)
- added R14: 470K, Resistor_SMD:R_0805_2012Metric, F.Cu at (-52.3, 61.9)
- added R15: 1.5K, Resistor_SMD:R_0805_2012Metric, F.Cu at (-55.7, 63.8)
- added R16: 820K, Resistor_SMD:R_0805_2012Metric, F.Cu at (-55.7, 61.9)
- added R17: 1K, Resistor_SMD:R_0805_2012Metric, F.Cu at (-29.8, 39.0)
- added R18: 15K, Resistor_SMD:R_0805_2012Metric, F.Cu at (-64.9, 72.1)
- added R19: 1K, Resistor_SMD:R_0805_2012Metric, F.Cu at (-26.7, 36.5)
- added R2: 4.7K, Resistor_SMD:R_0805_2012Metric, F.Cu at (-74.9, 78.6)
- added R3: 10K, Resistor_SMD:R_0805_2012Metric, F.Cu at (-33.2, 39.0)
- added R4: 10K, Resistor_SMD:R_0805_2012Metric, F.Cu at (-33.2, 41.0)
- added R5: 10K, Resistor_SMD:R_0805_2012Metric, F.Cu at (-71.5, 78.6)
- added R6: 10K, Resistor_SMD:R_0805_2012Metric, F.Cu at (-60.8, 67.3)
- added R7: 10K, Resistor_SMD:R_0805_2012Metric, F.Cu at (-68.3, 71.2)
- added R8: 10K, Resistor_SMD:R_0805_2012Metric, F.Cu at (-24.3, 33.7)
- added R9: 10K, Resistor_SMD:R_0805_2012Metric, F.Cu at (-68.1, 79.0)
- added SW1: Rotary_Encoder_Switch, Rotary_Encoder:RotaryEncoder_Alps_EC12E-Switch_Vertical_H20mm_CircularMountingHoles, F.Cu at (53.3, 51.7)
- added SW2: Rotary_Encoder_Switch, Rotary_Encoder:RotaryEncoder_Alps_EC12E-Switch_Vertical_H20mm_CircularMountingHoles, F.Cu at (78.5, 51.7)
- added SW3: Rotary_Encoder_Switch, Rotary_Encoder:RotaryEncoder_Alps_EC12E-Switch_Vertical_H20mm_CircularMountingHoles, F.Cu at (103.8, 51.7)
- added SW4: Rotary_Encoder_Switch, Rotary_Encoder:RotaryEncoder_Alps_EC12E-Switch_Vertical_H20mm_CircularMountingHoles, F.Cu at (128.9, 51.7)
- added U1: AMS1117-3.3, Package_TO_SOT_SMD:SOT-223-3_TabPin2, F.Cu at (165.4, 27.4)
- added U3: ILI9341, Connector_PinHeader_2.54mm:PinHeader_1x18_P2.54mm_Horizontal, F.Cu at (-82.9, 32.6)
- added U4: MCP602, Package_SO:SOIC-8_3.9x4.9mm_P1.27mm, F.Cu at (-61.1, 63.6)
- renumbered C1 to C3, C2 to C4, C3 to C5, C4 to C6, C5 to C7, C6 to C8, C7 to C9, D6 to D10, D7 to D11, D8 to D12, D9 to D13, D10 to D14, D11 to D15, D12 to D16, D13 to D17, D14 to D18, D15 to D19, D16 to D20, D17 to D21, D18 to D22, D19 to D23, D20 to D24, D21 to D25, D22 to D26, D23 to D27, D24 to D28, D25 to D29, D26 to D30, D1 to D5, D2 to D6, D3 to D7, D4 to D8, D5 to D9, SW6 to SW10, SW7 to SW11, SW8 to SW12, SW9 to SW13, SW10 to SW14, SW11 to SW15, SW12 to SW16, SW13 to SW17, SW14 to SW18, SW15 to SW19, SW16 to SW20, SW17 to SW21, SW18 to SW22, SW19 to SW23, SW20 to SW24, SW21 to SW25, SW22 to SW26, SW23 to SW27, SW24 to SW28, SW25 to SW29, SW26 to SW30, SW1 to SW5, SW2 to SW6, SW3 to SW7, SW4 to SW8, SW5 to SW9, U1 to U2
Connections:
- D5 pad 1: COL1 -> COL5
- D6 pad 1: COL2 -> COL6
- J2 pad 6: SDA -> SCL
- J3 pad 3: SDA -> SCL
- U2 pad 42: Net-(U1-Pad42) -> SCL
- U2 pad 43: Net-(U1-Pad43) -> SCL
