File: OTTO-dac/OTTOdac.kicad_pcb (KiCad board)
At the start: 2 copper layers, 38.8 x 66.6 mm, 42 parts, among them J1 Conn_01x10, J2 Audio_IN, J3 Audio_OUT, J4 SJ1-42536-SMT, J5 Speaker, U1 AMS1117-3.3, U2 SGTL5000, U3 LM4860, X1 XO32

Commit message: mainboard
Parts:
- U1: footprint Package_TO_SOT_SMD:SOT-23 -> Package_TO_SOT_SMD:SOT-223-3_TabPin2
- moved U1 3.54 mm to (307.4, 124.0), turned to 0 degrees
Routing:
- net GNDREF: track 159.2 -> 165.2 mm
- net +3V3: track 59.8 -> 58.5 mm
- net Net-(C6-Pad1): track 22.4 -> 21.4 mm
Changed lines of the file:
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@@
     (thickness 1.6)
     (drawings 1354)
-    (tracks 304)
+    (tracks 311)
     (zones 0)
     (modules 42)
@@
   )
   (setup
-    (last_trace_width 0.22)
+    (last_trace_width 0.25)
     (user_trace_width 0.18)
     (user_trace_width 0.25)
@@
     )
   )
-  (module Package_TO_SOT_SMD:SOT-23 (layer F.Cu)
-    (at 305.383869 126.912758 180)
-    (descr "SOT-23, Standard")
-    (tags SOT-23)
-    (attr smd)
-    (fp_text reference U1 (at 0 -2.5 180) (layer F.SilkS)
-      (effects (font (size 1 1) (thickness 0.15)))
-    )
-    (fp_text value AMS1117-3.3 (at 0 2.5 180) (layer F.Fab)
-      (effects (font (size 1 1) (thickness 0.15)))
-    )
-    (fp_text user %R (at 0 0 270) (layer F.Fab)
-      (effects (font (size 0.5 0.5) (thickness 0.075)))
-    )
-    (fp_line (start -0.7 -0.95) (end -0.7 1.5) (layer F.Fab) (width 0.1))
-    (fp_line (start -0.15 -1.52) (end 0.7 -1.52) (layer F.Fab) (width 0.1))
-    (fp_line (start -0.7 -0.95) (end -0.15 -1.52) (layer F.Fab) (width 0.1))
-    (fp_line (start 0.7 -1.52) (end 0.7 1.52) (layer F.Fab) (width 0.1))
-    (fp_line (start -0.7 1.52) (end 0.7 1.52) (layer F.Fab) (width 0.1))
-    (fp_line (start 0.76 1.58) (end 0.76 0.65) (layer F.SilkS) (width 0.12))
-    (fp_line (start 0.76 -1.58) (end 0.76 -0.65) (layer F.SilkS) (width 0.12))
-    (fp_line (start -1.7 -1.75) (end 1.7 -1.75) (layer F.CrtYd) (width 0.05))
-    (fp_line (start 1.7 -1.75) (end 1.7 1.75) (layer F.CrtYd) (width 0.05))
-    (fp_line (start 1.7 1.75) (end -1.7 1.75) (layer F.CrtYd) (width 0.05))
-    (fp_line (start -1.7 1.75) (end -1.7 -1.75) (layer F.CrtYd) (width 0.05))
-    (fp_line (start 0.76 -1.58) (end -1.4 -1.58) (layer F.SilkS) (width 0.12))
-    (fp_line (start 0.76 1.58) (end -0.7 1.58) (layer F.SilkS) (width 0.12))
-    (pad 1 smd rect (at -1 -0.95 180) (size 0.9 0.8) (layers F.Cu F.Paste F.Mask)
-      (net 1 GNDREF))
-    (pad 2 smd rect (at -1 0.95 180) (size 0.9 0.8) (layers F.Cu F.Paste F.Mask)
-      (net 14 "Net-(C6-Pad1)"))
-    (pad 3 smd rect (at 1 0 180) (size 0.9 0.8) (layers F.Cu F.Paste F.Mask)
-      (net 3 +3V3))
-    (model ${KISYS3DMOD}/Package_TO_SOT_SMD.3dshapes/SOT-23.wrl
-      (at (xyz 0 0 0))
-      (scale (xyz 1 1 1))
-      (rotate (xyz 0 0 0))
-    )
-  )
   (module Sensor_Audio:QFN-32-NXP-SGTL5000 (layer F.Cu)
     (at 309.969713 105.886548 90)
@@
     (pad 1 np_thru_hole circle (at 0 0) (size 2.5 2.5) (drill 2.5) (layers *.Cu *.Mask))
   )
+  (module Package_TO_SOT_SMD:SOT-223-3_TabPin2 (layer F.Cu)
+    (at 307.428234 124.02262)
+    (descr "module CMS SOT223 4 pins")
+    (tags "CMS SOT")
+    (attr smd)
+    (fp_text reference U1 (at 0 -4.5) (layer F.SilkS)
+      (effects (font (size 1 1) (thickness 0.15)))
+    )
+    (fp_text value AMS1117-3.3 (at 0 4.5) (layer F.Fab)
+      (effects (font (size 1 1) (thickness 0.15)))
+    )
+    (fp_text user %R (at 0 0 90) (layer F.Fab)
+      (effects (font (size 0.8 0.8) (thickness 0.12)))
+    )
+    (fp_line (start 1.91 3.41) (end 1.91 2.15) (layer F.SilkS) (width 0.12))
+    (fp_line (start 1.91 -3.41) (end 1.91 -2.15) (layer F.SilkS) (width 0.12))
+    (fp_line (start 4.4 -3.6) (end -4.4 -3.6) (layer F.CrtYd) (width 0.05))
+    (fp_line (start 4.4 3.6) (end 4.4 -3.6) (layer F.CrtYd) (width 0.05))
+    (fp_line (start -4.4 3.6) (end 4.4 3.6) (layer F.CrtYd) (width 0.05))
+    (fp_line (start -4.4 -3.6) (end -4.4 3.6) (layer F.CrtYd) (width 0.05))
+    (fp_line (start -1.85 -2.35) (end -0.85 -3.35) (layer F.Fab) (width 0.1))
+    (fp_line (start -1.85 -2.35) (end -1.85 3.35) (layer F.Fab) (width 0.1))
+    (fp_line (start -1.85 3.41) (end 1.91 3.41) (layer F.SilkS) (width 0.12))
+    (fp_line (start -0.85 -3.35) (end 1.85 -3.35) (layer F.Fab) (width 0.1))
+    (fp_line (start -4.1 -3.41) (end 1.91 -3.41) (layer F.SilkS) (width 0.12))
+    (fp_line (start -1.85 3.35) (end 1.85 3.35) (layer F.Fab) (width 0.1))
+    (fp_line (start 1.85 -3.35) (end 1.85 3.35) (layer F.Fab) (width 0.1))
+    (pad 2 smd rect (at 3.15 0) (size 2 3.8) (layers F.Cu F.Paste F.Mask)
+      (net 14 "Net-(C6-Pad1)"))
+    (pad 2 smd rect (at -3.15 0) (size 2 1.5) (layers F.Cu F.Paste F.Mask)
+      (net 14 "Net-(C6-Pad1)"))
+    (pad 3 smd rect (at -3.15 2.3) (size 2 1.5) (layers F.Cu F.Paste F.Mask)
+      (net 3 +3V3))
+    (pad 1 smd rect (at -3.15 -2.3) (size 2 1.5) (layers F.Cu F.Paste F.Mask)
+      (net 1 GNDREF))
+    (model ${KISYS3DMOD}/Package_TO_SOT_SMD.3dshapes/SOT-223.wrl
+      (at (xyz 0 0 0))
+      (scale (xyz 1 1 1))
+      (rotate (xyz 0 0 0))
+    )
+  )
   (gr_line (start 319.928234 120.923074) (end 319.928234 86.423074) (layer Cmts.User) (width 0.2))
   (gr_line (start 297.428234 86.423074) (end 319.928234 86.423074) (layer Cmts.User) (width 0.2))
@@
   (segment (start 329.428234 146.023074) (end 331.081577 146.023074) (width 0.4) (layer F.Cu) (net 1))
   (segment (start 331.081577 146.023074) (end 332.433869 144.670782) (width 0.4) (layer F.Cu) (net 1))
+  (segment (start 301.128234 125.690347) (end 301.128234 126.277847) (width 0.25) (layer F.Cu) (net 1))
+  (segment (start 301.128234 124.62262) (end 301.128234 125.690347) (width 0.25) (layer F.Cu) (net 1))
+  (segment (start 304.028234 121.72262) (end 301.128234 124.62262) (width 0.25) (layer F.Cu) (net 1))
+  (segment (start 304.278234 121.72262) (end 304.028234 121.72262) (width 0.25) (layer F.Cu) (net 1))
   (segment (start 309.568868 131.105259) (end 309.633869 131.040258) (width 0.4) (layer F.Cu) (net 2))
   (segment (start 309.568868 134.062757) (end 309.568868 131.105259) (width 0.4) (layer F.Cu) (net 2))
@@
   (segment (start 309.633869 129.572758) (end 310.835845 129.572758) (width 0.6) (layer B.Cu) (net 2))
   (segment (start 310.835845 129.572758) (end 315.425845 134.162758) (width 0.6) (layer B.Cu) (net 2))
-  (segment (start 296.928234 128.152847) (end 301.128234 128.152847) (width 0.22) (layer F.Cu) (net 3))
+  (segment (start 296.928234 128.152847) (end 301.128234 128.152847) (width 0.25) (layer F.Cu) (net 3))
   (segment (start 310.219713 103.486548) (end 310.219713 100.036547) (width 0.22) (layer F.Cu) (net 3))
   (segment (start 308.326708 112.554373) (end 308.328234 112.552847) (width 0.22) (layer F.Cu) (net 3))
@@
   (segment (start 305.922214 88.839047) (end 304.319714 87.236547) (width 0.22) (layer F.Cu) (net 3))
   (segment (start 305.922214 90.636547) (end 305.922214 88.839047) (width 0.22) (layer F.Cu) (net 3))
-  (segment (start 302.368323 126.912758) (end 304.383869 126.912758) (width 0.22) (layer F.Cu) (net 3))
-  (segment (start 301.128234 128.152847) (end 302.368323 126.912758) (width 0.22) (layer F.Cu) (net 3))
-  (segment (start 308.326708 116.352847) (end 308.326708 115.552847) (width 0.22) (layer F.Cu) (net 3))
-  (segment (start 308.326708 125.719919) (end 308.326708 116.352847) (width 0.22) (layer F.Cu) (net 3))
-  (segment (start 304.383869 126.912758) (end 307.133869 126.912758) (width 0.22) (layer F.Cu) (net 3))
-  (segment (start 307.133869 126.912758) (end 308.326708 125.719919) (width 0.22) (layer F.Cu) (net 3))
   (via (at 307.433869 111.170782) (size 0.6) (drill 0.3) (layers F.Cu B.Cu) (net 3))
   (segment (start 308.328234 112.552847) (end 308.328234 112.065147) (width 0.22) (layer F.Cu) (net 3))
@@
   (segment (start 305.922214 97.659127) (end 308.183869 99.920782) (width 0.22) (layer F.Cu) (net 3))
   (segment (start 305.922214 94.636547) (end 305.922214 97.659127) (width 0.22) (layer F.Cu) (net 3))
+  (segment (start 304.278234 127.32262) (end 304.278234 126.32262) (width 0.25) (layer F.Cu) (net 3))
+  (segment (start 303.448007 128.152847) (end 304.278234 127.32262) (width 0.25) (layer F.Cu) (net 3))
+  (segment (start 301.128234 128.152847) (end 303.448007 128.152847) (width 0.25) (layer F.Cu) (net 3))
+  (segment (start 308.326708 116.352847) (end 308.326708 115.552847) (width 0.25) (layer F.Cu) (net 3))
+  (segment (start 308.326708 122.524146) (end 308.326708 116.352847) (width 0.25) (layer F.Cu) (net 3))
+  (segment (start 304.528234 126.32262) (end 308.326708 122.524146) (width 0.25) (layer F.Cu) (net 3))
+  (segment (start 304.278234 126.32262) (end 304.528234 126.32262) (width 0.25) (layer F.Cu) (net 3))
   (segment (start 324.482214 137.927976) (end 324.426708 137.87247) (width 0.22) (layer F.Cu) (net 4))
   (segment (start 324.482214 142.836547) (end 324.482214 137.927976) (width 0.22) (layer F.Cu) (net 4))
@@
   (segment (start 305.482214 110.236547) (end 305.082214 109.836547) (width 0.22) (layer F.Cu) (net 14))
   (segment (start 305.882214 110.236547) (end 305.482214 110.236547) (width 0.22) (layer F.Cu) (net 14))
-  (segment (start 306.383869 125.962758) (end 306.383869 110.738202) (width 0.22) (layer F.Cu) (net 14))
   (segment (start 306.383869 110.738202) (end 305.882214 110.236547) (width 0.22) (layer F.Cu) (net 14))
+  (segment (start 306.383869 122.166985) (end 306.383869 110.738202) (width 0.25) (layer F.Cu) (net 14))
+  (segment (start 304.528234 124.02262) (end 306.383869 122.166985) (width 0.25) (layer F.Cu) (net 14))
+  (segment (start 304.278234 124.02262) (end 304.528234 124.02262) (width 0.25) (layer F.Cu) (net 14))
   (segment (start 313.482214 112.581827) (end 313.453234 112.552847) (width 0.22) (layer F.Cu) (net 15))
   (segment (start 313.453234 115.552847) (end 313.482214 115.523867) (width 0.22) (layer F.Cu) (net 15))
