File: OTTO-power/OTTO-power.kicad_pcb (KiCad board)
At the start: 2 copper layers, 72.5 x 23.5 mm, 43 parts, among them J1 Barrel_Jack, J2 Conn_01x10, J3 USB_B_Micro, J4 battery, SW1 SW_Push, U1 MAX8903A, U2 MAX17048, U3 TPS61090, U4 XC6210

Commit message: some rework on the routing
Parts:
- added REF**: MountingHole_2.2mm_M2_DIN965, MountingHole:MountingHole_2.2mm_M2_DIN965, F.Cu at (181.5, 38.8)
- added REF**: MountingHole_2.2mm_M2_DIN965, MountingHole:MountingHole_2.2mm_M2_DIN965, F.Cu at (193.5, 26.3)
- added REF**: MountingHole_2.2mm_M2_DIN965, MountingHole:MountingHole_2.2mm_M2_DIN965, F.Cu at (219.5, 44.8)
- added REF**: MountingHole_2.2mm_M2_DIN965, MountingHole:MountingHole_2.2mm_M2_DIN965, F.Cu at (152.0, 44.8)
- moved L2 1.24 mm to (157.0, 43.6)
- moved C9 1.20 mm to (158.2, 38.6)
- moved C10 0.65 mm to (162.7, 43.6)
Routing:
- net SYS: track 6.27 -> 14.9 mm, vias 3 -> 8
- net GNDA: track 0.58 -> 6.84 mm, vias 0 -> 2
- net CHG_OUT: track 48.7 -> 54.3 mm, vias 1 -> 3
- net OUT_PIN: track 17.8 -> 18.3 mm, vias 0 -> 1
- added copper zone on F.Cu, net 5V
- added copper zone on F.Cu, net GNDA
